File: RP2040_ESP32_dual_ESC/ESC1.kicad_sch (KiCad schematic)
At the start: 40 parts, among them J1 A, J2 B, J3 C, Q1 HYG025N06LS1C2, Q2 HYG025N06LS1C2, Q3 HYG025N06LS1C2, Q4 HYG025N06LS1C2, Q5 HYG025N06LS1C2, Q6 HYG025N06LS1C2, U1 LM324, U2 LM5109BMA, U3 LM5109BMA, U4 LM5109BMA

Commit message: t
Parts:
- R11, R12: footprint (none) -> Resistor_SMD:R_0603_1608Metric; LCSC (none) -> C21189
- R15, R16: footprint (none) -> Resistor_SMD:R_0603_1608Metric; LCSC (none) -> C25804
- R27: renamed from R10; footprint (none) -> Resistor_SMD:R_0603_1608Metric; LCSC (none) -> C21189
- R3: footprint (none) -> Resistor_SMD:R_1206_3216Metric
- R39: renamed from R14; footprint (none) -> Resistor_SMD:R_0603_1608Metric; LCSC (none) -> C25804
- renumbered C2 to C24, C4 to C25, C6 to C27, C7 to C29, D1 to D6, D2 to D7, D3 to D8, J1 to J4, J2 to J5, J3 to J6, Q4 to Q10, Q5 to Q11, Q6 to Q12, Q1 to Q7, Q2 to Q8, Q3 to Q9, R1 to R19, R2 to R20, R4 to R22, R5 to R23, R7 to R24, R8 to R25, R9 to R26, R13 to R38, R17 to R42, R18 to R43, U3 to U10, U4 to U11, U1 to U8, U2 to U9
Connections:
- net HB2: now reaches C25.1, D7.1 (K), U10.8 (HB)
- net gate_H2: now reaches Q9.3 (G), R26.2
- net HO2: now reaches R26.1, U10.7 (HO)
- net gate_L3: now reaches Q12.3 (G), R43.2
- net LO2: now reaches R38.1, U10.5 (LO)
- net gate_L2: now reaches Q10.3 (G), R38.2
- net HB1: now reaches C24.1, D6.1 (K), U9.8 (HB)
- net LO3: now reaches R43.1, U11.5 (LO)
- net LO1: now reaches R25.1, U9.5 (LO)
- net gate_L1: now reaches Q8.3 (G), R25.2
- net HO1: now reaches R22.1, U9.7 (HO)
- net gate_H1: now reaches Q7.3 (G), R22.2
- net HB3: now reaches C27.1, D8.1 (K), U11.8 (HB)
- net gate_H3: now reaches Q11.3 (G), R42.2
- net HO3: now reaches R42.1, U11.7 (HO)
Other:
- moved on the sheet: R19, R20, R23, R24
