File: RP2040_ESP32_dual_ESC/RP2040.kicad_sch (KiCad schematic)
At the start: 36 parts, among them J7 pins, SW1 SW_SPST, U5 LM4040DBZ-3.0, U6 W25Q128JVS, U7 RP2040, Y1 ABLS-12.000MHZ-B4-T

Commit message: t
Parts:
- removed FID1: Fiducial, Z_mycustom_footprint_lib:10x10_cm, symbol Mechanical:Fiducial
Changed lines of the file:
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@@
     (pin "2")
-  )
-  (symbol (lib_id "Mechanical:Fiducial") (at 22.86 105.41 0) (unit 1)
-    (in_bom no) (on_board yes) (fields_autoplaced)
-    (property "Reference" "FID1" (id 0) (at 25.4 104.1399 0)
-      (effects (font (size 1.27 1.27)) (justify left))
-    )
-    (property "Value" "Fiducial" (id 1) (at 25.4 106.6799 0)
-      (effects (font (size 1.27 1.27)) (justify left))
-    )
-    (property "Footprint" "Z_mycustom_footprint_lib:10x10_cm" (id 2) (at 22.86 105.41 0)
-      (effects (font (size 1.27 1.27)) hide)
-    )
-    (property "Datasheet" "~" (id 3) (at 22.86 105.41 0)
-      (effects (font (size 1.27 1.27)) hide)
-    )
   )
   (symbol (lib_id "power:GND") (at 46.99 166.37 0) (mirror y) (unit 1)
