File: RP2040_ESP32_dual_ESC/RP2040_ESP32_dual_ESC.kicad_pcb (KiCad board)
At the start: 2 copper layers, 100 x 100 mm, 92 parts, among them J1 A, J2 B, J3 C, J4 A, J5 B, J6 C, J7 pins, Q1 HYG025N06LS1C2, Q10 HYG025N06LS1C2, Q11 HYG025N06LS1C2, Q12 HYG025N06LS1C2, Q2 HYG025N06LS1C2, Q3 HYG025N06LS1C2, Q4 HYG025N06LS1C2, Q5 HYG025N06LS1C2, Q6 HYG025N06LS1C2, Q7 HYG025N06LS1C2, Q8 HYG025N06LS1C2, Q9 HYG025N06LS1C2, SW1 SW_SPST, U1 LM324, U10 LM5109BMA, U11 LM5109BMA, U2 LM5109BMA, U3 LM5109BMA, U4 LM5109BMA, U5 LM4040DBZ-3.0, U6 W25Q128JVS, U7 RP2040, U8 LM324, U9 LM5109BMA, Y1 ABLS-12.000MHZ-B4-T

Commit message: t
Parts:
- removed FID1: Fiducial, Z_mycustom_footprint_lib:10x10_cm
- added R10: 0, Resistor_SMD:R_0603_1608Metric, F.Cu at (88.0, 134.0)
- added R11: 0, Resistor_SMD:R_0603_1608Metric, F.Cu at (104.8, 134.0)
- added R12: 0, Resistor_SMD:R_0603_1608Metric, F.Cu at (121.4, 134.2)
- added R14: 10K, Resistor_SMD:R_0603_1608Metric, F.Cu at (108.0, 129.2)
- added R15: 10K, Resistor_SMD:R_0603_1608Metric, F.Cu at (106.5, 129.2)
- added R16: 10K, Resistor_SMD:R_0603_1608Metric, F.Cu at (109.7, 129.2)
- added R21: 5m, Resistor_SMD:R_1206_3216Metric, F.Cu at (204.1, 100.6)
- added R27: 0, Resistor_SMD:R_0603_1608Metric, F.Cu at (185.9, 138.4)
- added R28: 0, Resistor_SMD:R_0603_1608Metric, F.Cu at (185.9, 135.9)
- added R29: 0, Resistor_SMD:R_0603_1608Metric, F.Cu at (189.9, 135.9)
- added R3: 5m, Resistor_SMD:R_1206_3216Metric, F.Cu at (209.2, 105.8)
- added R39: 10K, Resistor_SMD:R_0603_1608Metric, F.Cu at (181.2, 118.5)
- added R40: 10K, Resistor_SMD:R_0603_1608Metric, F.Cu at (185.2, 116.0)
- added R41: 10K, Resistor_SMD:R_0603_1608Metric, F.Cu at (181.2, 116.0)
- C1, C3, C5: moved to B.Cu
- moved U1 87.3 mm to (107.9, 123.0), turned to -90 degrees
- moved Q12 70.7 mm to (268.1, 109.1)
- moved Q11 65.8 mm to (268.4, 100.9)
- moved Q9 58.6 mm to (235.9, 123.6)
- moved Q10 58.1 mm to (235.9, 131.8)
- moved J5 55.4 mm to (230.7, 129.9)
- moved J6 54.6 mm to (263.0, 107.2)
- moved Q8 39.1 mm to (227.2, 107.7)
- moved J4 34.3 mm to (222.1, 106.1)
- moved Q7 30.7 mm to (227.2, 99.5)
- moved R26 30.3 mm to (214.8, 75.2)
- moved R38 30.3 mm to (218.8, 75.2)
- moved R18 27.2 mm to (120.3, 136.0), turned to 0 degrees
- moved C6 25.0 mm to (116.8, 134.4), turned to 180 degrees
- moved R17 24.5 mm to (115.9, 136.0), turned to 180 degrees
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Connections:
- net Net-(C2-Pad1) renamed /ESC2/HB1
- net Net-(C24-Pad1) renamed /ESC1/HB1
- net Net-(C25-Pad1) renamed /ESC1/HB2
- net Net-(C27-Pad1) renamed /ESC1/HB3
- net Net-(C4-Pad1) renamed /ESC2/HB2
- net Net-(C6-Pad1) renamed /ESC2/HB3
- net Net-(Q1-Pad3) renamed /ESC2/gate_H1
- net Net-(Q10-Pad3) renamed /ESC1/gate_L2
- net Net-(Q11-Pad3) renamed /ESC1/gate_H3
- net Net-(Q12-Pad3) renamed /ESC1/gate_L3
- net Net-(Q2-Pad3) renamed /ESC2/gate_L1
- net Net-(Q3-Pad3) renamed /ESC2/gate_H2
- net Net-(Q4-Pad3) renamed /ESC2/gate_L2
- net Net-(Q5-Pad3) renamed /ESC2/gate_H3
- net Net-(Q6-Pad3) renamed /ESC2/gate_L3
- net Net-(Q7-Pad3) renamed /ESC1/gate_H1
- net Net-(Q8-Pad3) renamed /ESC1/gate_L1
- net Net-(Q9-Pad3) renamed /ESC1/gate_H2
- net Net-(R13-Pad1) renamed /ESC2/LO2
- net Net-(R17-Pad1) renamed /ESC2/HO3
- net Net-(R18-Pad1) renamed /ESC2/LO3
- net Net-(R22-Pad1) renamed /ESC1/HO1
- net Net-(R25-Pad1) renamed /ESC1/LO1
- net Net-(R26-Pad1) renamed /ESC1/HO2
- net Net-(R38-Pad1) renamed /ESC1/LO2
- net Net-(R4-Pad1) renamed /ESC2/HO1
- net Net-(R42-Pad1) renamed /ESC1/HO3
- net Net-(R43-Pad1) renamed /ESC1/LO3
- net Net-(R8-Pad1) renamed /ESC2/LO1
- net Net-(R9-Pad1) renamed /ESC2/HO2
Routing:
- net /ESC2/B1: track 0.00 -> 28.8 mm
- net /ESC2/A1: track 0.00 -> 27.7 mm
- net Net-(R12-Pad1): track 0.00 -> 27.4 mm, vias 0 -> 4
- net Net-(R10-Pad1): track 0.00 -> 25.6 mm, vias 0 -> 2
- net /ESC2/C1: track 0.00 -> 25.3 mm
- net /ESC2/star2: track 0.00 -> 19.4 mm
- net +15V: track 0.00 -> 16.4 mm, vias 0 -> 3
- net Net-(R11-Pad1): track 0.00 -> 9.95 mm, vias 0 -> 2
- net GND: track 0.00 -> 9.87 mm, vias 0 -> 4
- net /ESC2/LO2: track 0.00 -> 8.89 mm, vias 0 -> 2
- net /ESC2/LO1: track 0.00 -> 8.01 mm, vias 0 -> 2
- net /ESC2/LO3: track 0.00 -> 7.90 mm, vias 0 -> 2
- net /ESC2/HB3: track 0.00 -> 4.78 mm
- net /ESC2/HB1: track 0.00 -> 4.78 mm
- net /ESC2/HB2: track 0.00 -> 4.70 mm
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- added copper zone on F.Cu, net /ESC2/A1
Other:
- board outline removed
