File: ESP32_dual_ESC/ESP32_dual_ESC.kicad_pcb (KiCad board)
At the start: 4 copper layers, 100 x 100 mm, 136 parts, among them J1 A, J10 Conn_01x04, J11 A, J12 B, J13 C, J2 B, J3 C, J4 pins, J5 Conn_01x04, J6 USB_C_Receptacle, J7 Conn_01x06, J8 Conn_01x06, J9 Conn_01x04, Q1 HYG025N06LS1C2, Q10 HYG025N06LS1C2, Q11 HYG025N06LS1C2, Q12 HYG025N06LS1C2, Q13 N MOSFET, Q2 HYG025N06LS1C2, Q3 HYG025N06LS1C2, Q4 HYG025N06LS1C2, Q5 HYG025N06LS1C2, Q6 HYG025N06LS1C2, Q7 HYG025N06LS1C2, Q8 HYG025N06LS1C2, Q9 HYG025N06LS1C2, SW1 MCU_RESET, SW2 MCU_RESET, SW3 MCU_RESET, U1 LM324, U10 LM324, U11 DRV8300N, U12 INA219AxD, U2 LM5109BMA, U3 LM5109BMA, U4 LM5109BMA, U5 W25Q128JVS, U6 ESP32-S3-WROOM-1, U7 SRV05-4, U8 MCP6002-xSN, U9 CJ431

Commit message: g
Parts:
- removed C23: 10u, Capacitor_SMD:C_0603_1608Metric
- removed C8: 100n, Capacitor_SMD:C_0603_1608Metric
- removed J4: pins, Connector_PinHeader_2.54mm:PinHeader_1x02_P2.54mm_Vertical
- removed J5, J9: Conn_01x04, Connector_PinHeader_2.54mm:PinHeader_1x04_P2.54mm_Vertical
- removed J8: Conn_01x06, Connector_PinHeader_2.54mm:PinHeader_1x06_P2.54mm_Vertical
- removed Q13: N MOSFET, Package_DFN_QFN:PQFN-8-EP_6x5mm_P1.27mm_Generic
- removed R27: 10k, Resistor_SMD:R_0603_1608Metric
- removed SW2: MCU_RESET, SamacSys_Parts:PTS526SK15SMTR2LFS
- removed U5: W25Q128JVS, Package_SO:SOIC-8_5.23x5.23mm_P1.27mm
- removed U8: MCP6002-xSN, Package_SO:SOIC-8_3.9x4.9mm_P1.27mm
- added C66: 10u, Capacitor_SMD:C_1206_3216Metric, F.Cu at (131.3, 88.0)
- added C67: 10u, Capacitor_SMD:C_1206_3216Metric, F.Cu at (128.8, 88.0)
- added C68: 10u, Capacitor_SMD:C_1206_3216Metric, F.Cu at (131.4, 99.9)
- added C69: 10u, Capacitor_SMD:C_1206_3216Metric, F.Cu at (128.8, 99.9)
- added C7: 100n, Capacitor_SMD:C_0603_1608Metric, F.Cu at (115.9, 121.0)
- added C70: 10u, Capacitor_SMD:C_1206_3216Metric, F.Cu at (131.4, 112.0)
- added C71: 10u, Capacitor_SMD:C_1206_3216Metric, F.Cu at (128.8, 111.9)
- added C72: 10u, Capacitor_SMD:C_1206_3216Metric, F.Cu at (68.1, 89.8)
- added C73: 10u, Capacitor_SMD:C_1206_3216Metric, F.Cu at (70.6, 89.9)
- added C74: 10u, Capacitor_SMD:C_1206_3216Metric, F.Cu at (68.1, 101.7)
- added C75: 10u, Capacitor_SMD:C_1206_3216Metric, F.Cu at (70.5, 101.7)
- added C76: 10u, Capacitor_SMD:C_1206_3216Metric, F.Cu at (68.1, 113.6)
- added C77: 10u, Capacitor_SMD:C_1206_3216Metric, F.Cu at (70.6, 113.6)
- added C78: 1u, Capacitor_SMD:C_0402_1005Metric, F.Cu at (121.8, 133.5)
- added D14: 1N5819WS, Diode_SMD:D_SOD-323, F.Cu at (126.9, 104.0)
- added D15: 1N5819WS, Diode_SMD:D_SOD-323, F.Cu at (126.9, 116.0)
- added D16: 1N5819WS, Diode_SMD:D_SOD-323, F.Cu at (72.8, 115.3)
- added D17: 1N5819WS, Diode_SMD:D_SOD-323, F.Cu at (72.8, 111.5)
- added D18: 1N5819WS, Diode_SMD:D_SOD-323, F.Cu at (72.8, 103.7)
- added D19: 1N5819WS, Diode_SMD:D_SOD-323, F.Cu at (72.7, 99.7)
- added D20: 1N5819WS, Diode_SMD:D_SOD-323, F.Cu at (72.8, 91.9)
- added D21: 1N5819WS, Diode_SMD:D_SOD-323, F.Cu at (72.8, 87.9)
- added J14: A, MountingHole:MountingHole_2.5mm_Pad_TopBottom, F.Cu at (95.0, 144.4)
- added J15: A, MountingHole:MountingHole_2.5mm_Pad_TopBottom, F.Cu at (105.0, 144.4)
- added Q20: MMBT5551L, Package_TO_SOT_SMD:SOT-23, F.Cu at (112.7, 57.4)
- added Q21: MMBT5551L, Package_TO_SOT_SMD:SOT-23, F.Cu at (111.3, 60.9)
- added R1: 10K, Resistor_SMD:R_0603_1608Metric, F.Cu at (97.0, 118.9)
- added R39: 22, Resistor_SMD:R_0603_1608Metric, F.Cu at (124.3, 115.2)
- added R4: 10K, Resistor_SMD:R_0603_1608Metric, F.Cu at (95.5, 118.0)
- added R42: 22, Resistor_SMD:R_0603_1608Metric, F.Cu at (75.3, 114.5)
- added R59: 22, Resistor_SMD:R_0603_1608Metric, F.Cu at (75.3, 112.4)
- added R60: 22, Resistor_SMD:R_0603_1608Metric, F.Cu at (75.3, 102.9)
- added R61: 22, Resistor_SMD:R_0603_1608Metric, F.Cu at (75.2, 100.6)
- added R62: 22, Resistor_SMD:R_0603_1608Metric, F.Cu at (75.3, 91.0)
- added R63: 22, Resistor_SMD:R_0603_1608Metric, F.Cu at (75.3, 88.7)
- added R64: 1k, Resistor_SMD:R_0402_1005Metric, F.Cu at (111.5, 133.9)
- added R65: 75k, Resistor_SMD:R_0402_1005Metric, F.Cu at (113.5, 133.9)
- added R66: 1k, Resistor_SMD:R_0402_1005Metric, F.Cu at (112.0, 135.4)
- added R67: 75k, Resistor_SMD:R_0402_1005Metric, F.Cu at (113.5, 135.9)
- added U13: MCP6002-xSN, Package_SO:SOIC-8_3.9x4.9mm_P1.27mm, F.Cu at (119.0, 136.7)
- C15, C16: value 1u -> 10u; footprint Capacitor_SMD:C_0402_1005Metric -> Capacitor_SMD:C_0805_2012Metric
- C19, C2, C4, C6: footprint Capacitor_SMD:C_0603_1608Metric -> Capacitor_SMD:C_0805_2012Metric
- C21: value 10u -> 100n
- D10, D7, D8, D9: value green -> 1N5819WS; footprint LED_SMD:LED_0805_2012Metric -> Diode_SMD:D_SOD-323
- J1, J11, J12, J13, J2, J3: footprint Mounting_Wuerth:Mounting_Wuerth_WA-SMSI-M1.6_H1.5mm_9774015633 -> MountingHole:MountingHole_2.5mm_Pad_TopBottom
- R18: value DNF -> 10k; footprint Resistor_SMD:R_0603_1608Metric_Pad0.98x0.95mm_HandSolder -> Resistor_SMD:R_0603_1608Metric
- R19: value 1k -> 10k
- R25, R26: value 10k -> 10K
- R28, R29, R30, R31: value 1k -> 22; footprint Resistor_SMD:R_0805_2012Metric -> Resistor_SMD:R_0603_1608Metric
- R37: value 10k -> 22
- moved Q6 191.1 mm to (60.8, 87.2), turned to 90 degrees
- moved Q4 180.8 mm to (60.8, 98.9), turned to 90 degrees
- moved Q5 180.6 mm to (66.0, 92.7), turned to -90 degrees
- moved J1 176.4 mm to (55.3, 112.2), turned to 180 degrees
- moved J2 173.0 mm to (55.3, 100.2), turned to 180 degrees
- moved Q2 171.5 mm to (60.8, 110.7), turned to 90 degrees
- moved J3 171.2 mm to (55.3, 88.2), turned to 180 degrees
- moved Q3 170.9 mm to (66.0, 104.4), turned to -90 degrees
- moved C1 167.8 mm to (86.2, 117.8), turned to 180 degrees
- moved D1 166.9 mm to (82.0, 117.9)
- moved R16 165.4 mm to (75.3, 92.8), turned to 180 degrees
- moved C3 165.1 mm to (86.0, 106.0), turned to 180 degrees
- moved R17 164.4 mm to (75.3, 87.0), turned to 180 degrees
- moved D2 164.1 mm to (81.8, 106.2)
- moved C5 163.3 mm to (86.1, 94.1), turned to 180 degrees
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Connections:
- net /MCU/MISO renamed /MCU/GPIO_15
- C15 pad 1: GND -> /ESC_V2/HB2
- C15 pad 2: /MCU/SWITCH_EN -> /ESC_V2/B1
- C16 pad 1: GND -> /ESC_V2/HB3
- C16 pad 2: /MCU/SWITCH_EN -> /ESC_V2/C1
- C21 pad 1: /ESC_V2/HB2 -> GND
- C21 pad 2: /ESC_V2/B1 -> +3V3
- D10 pad 2: /MCU/W5500_LED1 -> /ESC_V2/gate_L1
- D6 pad 1: +BATT -> VDC
- D7 pad 2: /MCU/W5500_LED4 -> /ESC_V2/gate_H3
- D8 pad 2: /MCU/W5500_LED3 -> /ESC_V2/gate_H2
- D9 pad 2: /MCU/W5500_LED2 -> /ESC_V2/gate_H1
- J7 pad 1: +3V3 -> GND
- J7 pad 2: SS_EXT -> Net-(J7-Pin_2)
- J7 pad 3: CLK_EXT -> Net-(J7-Pin_3)
- J7 pad 4: MOSI_EXT -> /MCU/RST
- J7 pad 5: MISO_EXT -> /MCU/DTR
- J7 pad 6: GND -> +3V3
- Q1 pad 1: ESC2_VCC -> ESC1_VCC
- Q3 pad 1: ESC2_VCC -> ESC1_VCC
- Q5 pad 1: ESC2_VCC -> ESC1_VCC
- R11 pad 1: Net-(U1B-+) -> Net-(U1A-+)
- R15 pad 2: Net-(U1B-+) -> Net-(U1A-+)
- R18 pad 1: +3V3 -> /MCU/DTR
- R18 pad 2: /MCU/QSPI_SS -> Net-(Q20-B)
- R19 pad 1: /MCU/QSPI_SS -> /MCU/RST
- R19 pad 2: /MCU/~{USB_BOOT} -> Net-(Q21-B)
- R25 pad 1: +3V3 -> +15V
- R25 pad 2: /MCU/Rail_V -> Net-(U10B-+)
- R26 pad 1: /MCU/Rail_V -> ESC2_VCC
- R26 pad 2: GND -> Net-(U10B--)
- R28 pad 1: Net-(D7-K) -> /ESC_V2/HO3
- R28 pad 2: GND -> Net-(D7-K)
- R29 pad 1: Net-(D8-K) -> /ESC_V2/HO2
- R29 pad 2: GND -> Net-(D8-K)
- R3 pad 1: VCC -> +15V
- R3 pad 2: ESC2_VCC -> ESC1_VCC
- R30 pad 1: Net-(D9-K) -> /ESC_V2/HO1
- R30 pad 2: GND -> Net-(D9-K)
- R31 pad 1: Net-(D10-K) -> /ESC_V2/LO1
- R31 pad 2: GND -> Net-(D10-K)
- R37 pad 1: /MCU/SWITCH_EN -> /ESC_V2/LO2
- R37 pad 2: +3V3 -> Net-(D14-K)
- R41 pad 1: VCC -> +15V
- R49 pad 1: Net-(U10B-+) -> Net-(U10A-+)
- R53 pad 2: Net-(U10B-+) -> Net-(U10A-+)
- R56 pad 1: VCC -> +15V
- R57 pad 1: VCC -> +15V
- SW3 pad 1: /MCU/ESP_BOOT -> GND
- SW3 pad 2: GND -> /MCU/ESP_BOOT
- U1 pad 1: /ESC_V1/Current_Out -> /MCU/GPIO_17
- U1 pad 14: /MCU/GPIO6 -> /MCU/GPIO_16
- U1 pad 2: Net-(U1A--) -> /ESC_V1/star2
- U1 pad 6: /ESC_V1/star2 -> Net-(U1B--)
- U1 pad 7: /MCU/GPIO8 -> /MCU/GPIO_08
- U1 pad 8: /MCU/GPIO7 -> /MCU/GPIO_12
- U10 pad 1: /MCU/GPIO29_ADC3 -> /MCU/GPIO_21
- U10 pad 14: /MCU/GPIO16 -> /MCU/GPIO_42
- U10 pad 2: Net-(U10A--) -> /ESC_V2/star2
- U10 pad 6: /ESC_V2/star2 -> Net-(U10B--)
- U10 pad 7: /MCU/GPIO18 -> /MCU/GPIO_11
- U10 pad 8: /MCU/GPIO17 -> /MCU/GPIO_14
- U11 pad 1: /MCU/GPIO10 -> /MCU/GPIO_39
- U11 pad 2: /MCU/GPIO12 -> /MCU/GPIO_37
- U11 pad 3: /MCU/GPIO14 -> /MCU/GPIO_36
- U11 pad 4: /MCU/GPIO11 -> /MCU/GPIO_35
- U11 pad 5: /MCU/GPIO13 -> /MCU/GPIO_40
- U11 pad 6: /MCU/GPIO15 -> /MCU/GPIO_41
- U12 pad 1: unconnected-(U12-A1-Pad1) -> GND
- U12 pad 2: unconnected-(U12-A0-Pad2) -> GND
- U2 pad 2: /MCU/GPIO0 -> /MCU/GPIO_18
- U2 pad 3: /MCU/GPIO1 -> /MCU/GPIO_13
- U3 pad 2: /MCU/GPIO2 -> /MCU/GPIO_04
- U3 pad 3: /MCU/GPIO3 -> /MCU/GPIO_05
- U4 pad 2: /MCU/GPIO4 -> /MCU/GPIO_06
- U4 pad 3: /MCU/GPIO5 -> /MCU/GPIO_07
- U6 pad 10: unconnected-(U6-GPIO17/U1TXD/ADC2_CH6-Pad10) -> /MCU/GPIO_17
- U6 pad 11: unconnected-(U6-GPIO18/U1RXD/ADC2_CH7/CLK_OUT3-Pad11) -> /MCU/GPIO_18
- U6 pad 12: unconnected-(U6-GPIO8/TOUCH8/ADC1_CH7/SUBSPICS1-Pad12) -> /MCU/GPIO_08
- U6 pad 17: unconnected-(U6-GPIO9/TOUCH9/ADC1_CH8/FSPIHD/SUBSPIHD-Pad17) -> current
- U6 pad 18: unconnected-(U6-GPIO10/TOUCH10/ADC1_CH9/FSPICS0/FSPIIO4/SUBSPICS0-Pad18) -> REF_2v5
- U6 pad 19: unconnected-(U6-GPIO11/TOUCH11/ADC2_CH0/FSPID/FSPIIO5/SUBSPID-Pad19) -> /MCU/GPIO_11
- U6 pad 20: unconnected-(U6-GPIO12/TOUCH12/ADC2_CH1/FSPICLK/FSPIIO6/SUBSPICLK-Pad20) -> /MCU/GPIO_12
- U6 pad 21: unconnected-(U6-GPIO13/TOUCH13/ADC2_CH2/FSPIQ/FSPIIO7/SUBSPIQ-Pad21) -> /MCU/GPIO_13
- U6 pad 22: unconnected-(U6-GPIO14/TOUCH14/ADC2_CH3/FSPIWP/FSPIDQS/SUBSPIWP-Pad22) -> /MCU/GPIO_14
- U6 pad 23: unconnected-(U6-GPIO21-Pad23) -> /MCU/GPIO_21
- U6 pad 24: unconnected-(U6-GPIO47/SPICLK_P/SUBSPICLK_P_DIFF-Pad24) -> /MCU/GPIO_47
- U6 pad 25: unconnected-(U6-GPIO48/SPICLK_N/SUBSPICLK_N_DIFF-Pad25) -> /MCU/GPIO_48
- U6 pad 28: unconnected-(U6-SPIIO6/GPIO35/FSPID/SUBSPID-Pad28) -> /MCU/GPIO_35
- U6 pad 29: unconnected-(U6-SPIIO7/GPIO36/FSPICLK/SUBSPICLK-Pad29) -> /MCU/GPIO_36
- U6 pad 30: unconnected-(U6-SPIDQS/GPIO37/FSPIQ/SUBSPIQ-Pad30) -> /MCU/GPIO_37
- U6 pad 31: unconnected-(U6-GPIO38/FSPIWP/SUBSPIWP-Pad31) -> /MCU/GPIO_38
- U6 pad 32: unconnected-(U6-MTCK/GPIO39/CLK_OUT3/SUBSPICS1-Pad32) -> /MCU/GPIO_39
- U6 pad 33: unconnected-(U6-MTDO/GPIO40/CLK_OUT2-Pad33) -> /MCU/GPIO_40
- U6 pad 34: unconnected-(U6-MTDI/GPIO41/CLK_OUT1-Pad34) -> /MCU/GPIO_41
- U6 pad 35: unconnected-(U6-MTMS/GPIO42-Pad35) -> /MCU/GPIO_42
- U6 pad 36: Net-(J5-Pin_2) -> Net-(J7-Pin_3)
- U6 pad 37: Net-(J5-Pin_3) -> Net-(J7-Pin_2)
- U6 pad 38: unconnected-(U6-GPIO2/TOUCH2/ADC1_CH1-Pad38) -> /MCU/GPIO_02
- U6 pad 39: unconnected-(U6-GPIO1/TOUCH1/ADC1_CH0-Pad39) -> /MCU/GPIO_01
- U6 pad 4: unconnected-(U6-GPIO4/TOUCH4/ADC1_CH3-Pad4) -> /MCU/GPIO_04
- U6 pad 5: unconnected-(U6-GPIO5/TOUCH5/ADC1_CH4-Pad5) -> /MCU/GPIO_05
- U6 pad 6: unconnected-(U6-GPIO6/TOUCH6/ADC1_CH5-Pad6) -> /MCU/GPIO_06
- U6 pad 7: unconnected-(U6-GPIO7/TOUCH7/ADC1_CH6-Pad7) -> /MCU/GPIO_07
- U6 pad 9: /MCU/SCLK -> /MCU/GPIO_16
Routing:
- net +3V3: track 0.00 -> 190.2 mm, vias 0 -> 6
- net +15V: track 0.00 -> 150.2 mm, vias 0 -> 4
- net REF_2v5: track 0.00 -> 86.6 mm, vias 0 -> 2
- net GND: track 0.00 -> 85.1 mm, vias 0 -> 238
- net current: track 0.00 -> 84.5 mm, vias 0 -> 2
- net /MCU/GPIO_11: track 0.00 -> 76.8 mm, vias 0 -> 2
- net /MCU/GPIO_14: track 0.00 -> 74.2 mm, vias 0 -> 2
- net /MCU/ESP_EN: track 0.00 -> 72.1 mm, vias 0 -> 3
- net /MCU/GPIO_42: track 0.00 -> 68.1 mm, vias 0 -> 2
- net /MCU/GPIO_21: track 0.00 -> 66.4 mm, vias 0 -> 4
- net /MCU/GPIO_08: track 0.00 -> 63.3 mm, vias 0 -> 4
- net /MCU/ESP_BOOT: track 0.00 -> 61.4 mm, vias 0 -> 3
- net /MCU/GPIO_18: track 0.00 -> 58.7 mm, vias 0 -> 2
- net /MCU/GPIO_17: track 0.00 -> 58.5 mm, vias 0 -> 2
- net /MCU/GPIO_13: track 0.00 -> 58.2 mm, vias 0 -> 2
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- added copper zone on F.Cu, net +15V
- added copper zone on B.Cu, net /ESC_V1/A1
- added copper zone on F.Cu, net /ESC_V1/A1
- added copper zone on In1.Cu, net /ESC_V1/A1
- added copper zone on In2.Cu, net /ESC_V1/A1
- added copper zone on B.Cu, net /ESC_V1/B1
- added copper zone on F.Cu, net /ESC_V1/B1
- added copper zone on In1.Cu, net /ESC_V1/B1
- added copper zone on In2.Cu, net /ESC_V1/B1
- added copper zone on B.Cu, net /ESC_V1/C1
- added copper zone on F.Cu, net /ESC_V1/C1
- added copper zone on In1.Cu, net /ESC_V1/C1
- added copper zone on In2.Cu, net /ESC_V1/C1
- added copper zone on B.Cu, net /ESC_V2/A1
- added copper zone on F.Cu, net /ESC_V2/A1
- added copper zone on In1.Cu, net /ESC_V2/A1
- added copper zone on In2.Cu, net /ESC_V2/A1
- added copper zone on B.Cu, net /ESC_V2/B1
- added copper zone on F.Cu, net /ESC_V2/B1
- added copper zone on In1.Cu, net /ESC_V2/B1
- added copper zone on In2.Cu, net /ESC_V2/B1
- added copper zone on B.Cu, net /ESC_V2/C1
- added copper zone on F.Cu, net /ESC_V2/C1
- added copper zone on In1.Cu, net /ESC_V2/C1
- added copper zone on In2.Cu, net /ESC_V2/C1
- added copper zone on B.Cu, net ESC1_VCC
- added copper zone on F.Cu, net ESC1_VCC
- added copper zone on B.Cu, net ESC2_VCC
- added copper zone on F.Cu, net ESC2_VCC
- added copper zone on B.Cu, net GND
- added copper zone on F.Cu, net GND
- added copper zone on In1.Cu, net GND
- added copper zone on In2.Cu, net GND
- added copper zone on B.Cu, net VDC
- added copper zone on F.Cu, net VDC

Commit message: l
Parts:
- added C23: 100u, Capacitor_SMD:CP_Elec_6.3x5.4, F.Cu at (137.0, 75.3)
- added C24: 1u, Capacitor_SMD:C_0402_1005Metric, F.Cu at (146.0, 67.2)
- added C26: 10u, Capacitor_SMD:C_0603_1608Metric, F.Cu at (147.2, 67.1)
- added C27: 1u, Capacitor_SMD:C_0402_1005Metric, F.Cu at (130.0, 76.3)
- added C28: 10u, Capacitor_SMD:C_0603_1608Metric, F.Cu at (131.3, 76.2)
- added C8: 100n, Capacitor_SMD:C_0603_1608Metric, F.Cu at (138.8, 62.5)
- added D22: B5819W_SL, Diode_SMD:D_SOD-123, F.Cu at (101.4, 83.1)
- added D23: B5819W_SL, Diode_SMD:D_SOD-123, F.Cu at (143.0, 63.2)
- added D24: B5819W_SL, Diode_SMD:D_SOD-123, F.Cu at (103.9, 83.1)
- added D25: green, LED_SMD:LED_0805_2012Metric, F.Cu at (101.8, 89.8)
- added J4: Conn_01x02, Connector_PinHeader_2.54mm:PinHeader_1x02_P2.54mm_Vertical, F.Cu at (147.0, 71.9)
- added JP2: Jumper_2_Bridged, Jumper:SolderJumper-2_P1.3mm_Bridged_RoundedPad1.0x1.5mm, F.Cu at (98.7, 92.2)
- added L1: 75u, Inductor_SMD:L_Changjiang_FNR8040S, F.Cu at (133.5, 65.3)
- added R2: 75k, Resistor_SMD:R_0402_1005Metric, F.Cu at (95.3, 116.5)
- added R27: 10K, Resistor_SMD:R_0603_1608Metric, F.Cu at (137.4, 70.8)
- added R40: 75k, Resistor_SMD:R_0402_1005Metric, F.Cu at (120.9, 122.4)
- added R44: 75k, Resistor_SMD:R_0402_1005Metric, F.Cu at (119.8, 120.9)
- added R6: 75k, Resistor_SMD:R_0402_1005Metric, F.Cu at (97.0, 117.5)
- added R68: 6.2k, Resistor_SMD:R_0603_1608Metric, F.Cu at (140.4, 70.8)
- added R69: 10K, Resistor_SMD:R_0603_1608Metric, F.Cu at (98.5, 89.7)
- added U5: TPS5430DDA, Package_SO:TI_SO-PowerPAD-8_ThermalVias, F.Cu at (141.6, 67.2)
- R1, R25, R26, R4: value 10K -> 1k; footprint Resistor_SMD:R_0603_1608Metric -> Resistor_SMD:R_0402_1005Metric
- R10, R11, R47, R48, R49, R9: value 0 -> 75k
- R12, R16, R17, R42, R5, R59, R60, R61, R62, R63, R7, R8: value 22 -> 56
- moved FID2 77.8 mm to (141.8, 124.9)
- moved FID3 51.9 mm to (138.0, 132.4)
- moved R17 29.2 mm to (75.3, 116.2), turned to 0 degrees
- moved R7 7.79 mm to (75.3, 102.8)
- moved R12 7.74 mm to (75.3, 91.1)
- moved FID1 6.50 mm to (59.0, 51.5)
- moved R16 5.81 mm to (75.3, 87.0)
- moved R8 5.75 mm to (75.2, 98.8)
- moved R5 5.56 mm to (75.3, 110.7)
- moved R1 1.78 mm to (95.5, 118.1), turned to -90 degrees
- moved R62 1.77 mm to (75.3, 92.8), turned to 0 degrees
- moved R4 1.75 mm to (97.0, 119.0), turned to -90 degrees
- moved R60 1.71 mm to (75.3, 104.6), turned to 0 degrees
- moved R32 1.20 mm to (115.6, 73.0)
- moved J10 0.94 mm to (118.8, 77.4)
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Connections:
- net Net-(J7-Pin_2) renamed /MCU/RX
- net Net-(J7-Pin_3) renamed /MCU/TX
- R1 pad 1: +15V -> Net-(U1B--)
- R1 pad 2: Net-(U1B-+) -> ESC1_VCC
- R12 pad 1: /ESC_V1/LO2 -> /ESC_V1/HO3
- R12 pad 2: /ESC_V1/gate_L2 -> Net-(D20-K)
- R16 pad 1: /ESC_V1/HO3 -> /ESC_V1/LO3
- R16 pad 2: /ESC_V1/gate_H3 -> /ESC_V1/gate_L3
- R17 pad 1: /ESC_V1/LO3 -> /ESC_V1/gate_H1
- R17 pad 2: /ESC_V1/gate_L3 -> /ESC_V1/HO1
- R25 pad 1: +15V -> Net-(U10B-+)
- R25 pad 2: Net-(U10B-+) -> +15V
- R26 pad 1: ESC2_VCC -> Net-(U10B--)
- R26 pad 2: Net-(U10B--) -> ESC2_VCC
- R4 pad 1: ESC1_VCC -> Net-(U1B-+)
- R4 pad 2: Net-(U1B--) -> +15V
- R5 pad 1: /ESC_V1/HO1 -> /ESC_V1/LO1
- R5 pad 2: /ESC_V1/gate_H1 -> /ESC_V1/gate_L1
- R59 pad 1: /ESC_V1/LO1 -> Net-(D17-K)
- R59 pad 2: Net-(D17-K) -> /ESC_V1/LO1
- R60 pad 1: /ESC_V1/HO2 -> /ESC_V1/gate_H2
- R60 pad 2: Net-(D18-K) -> /ESC_V1/HO2
- R61 pad 1: /ESC_V1/LO2 -> Net-(D19-K)
- R61 pad 2: Net-(D19-K) -> /ESC_V1/LO2
- R62 pad 1: /ESC_V1/HO3 -> /ESC_V1/gate_H3
- R62 pad 2: Net-(D20-K) -> /ESC_V1/HO3
- R63 pad 1: /ESC_V1/LO3 -> Net-(D21-K)
- R63 pad 2: Net-(D21-K) -> /ESC_V1/LO3
- R7 pad 1: /ESC_V1/LO1 -> /ESC_V1/HO2
- R7 pad 2: /ESC_V1/gate_L1 -> Net-(D18-K)
- R8 pad 1: /ESC_V1/HO2 -> /ESC_V1/LO2
- R8 pad 2: /ESC_V1/gate_H2 -> /ESC_V1/gate_L2
- U6 pad 38: /MCU/GPIO_02 -> SCL
- U6 pad 39: /MCU/GPIO_01 -> SDA
Routing:
- net SDA: track 0.00 -> 123.1 mm, vias 0 -> 7
- net SCL: track 0.00 -> 121.9 mm, vias 0 -> 6
- net +3V3: track 190.2 -> 276.2 mm, vias 6 -> 9
- net Net-(D22-K): track 0.00 -> 58.3 mm, vias 0 -> 2
- net +15V: track 150.2 -> 197.5 mm
- net +5V: track 17.5 -> 61.4 mm
- net GND: track 85.1 -> 108.1 mm, vias 238 -> 909
- net Net-(D23-K): track 0.00 -> 14.8 mm
- net Net-(U5-VSENSE): track 0.00 -> 3.11 mm
- net Net-(J4-Pin_2): track 0.00 -> 2.87 mm
- net Net-(JP2-B): track 0.00 -> 2.58 mm
- net /MCU/GPIO_15: track 2.34 -> 0.00 mm
- net Net-(U5-BOOT): track 0.00 -> 1.99 mm
- net /MCU/GPIO_17: track 58.5 -> 56.5 mm
- net /MCU/GPIO_18: track 58.7 -> 56.7 mm
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- added copper zone on F.Cu, net +3V3
Other:
- outline, holes or cut-outs redrawn
- board text added: "15V"
- board text added: "3V3"
- board text added: "5V"
- board text added: "A1"
- board text added: "B1"
- board text added: "BOOT"
- board text added: "C1"
- board text added: "DTR"
- board text added: "EN"
- board text added: "GND"
- board text added: "RST"
- board text added: "RX"
- board text added: "SCL"
- board text added: "SDA"
- board text added: "TX"
