File: ESP32_dual_ESC/MCU.kicad_sch (KiCad schematic)
At the start: 63 parts, among them J1 Conn_01x04, J2 Conn_01x06, J3 Conn_01x06, J4 USB_C_Receptacle, J4 pins, J5 Conn_01x04, J6 Conn_01x04, SW1 MCU_RESET, SW2 MCU_RESET, SW3 MCU_RESET, U1 ESP32-S3-WROOM-1, U10 MCP6002-xSN, U4 SRV05-4, U5 W25Q128JVS, U9 CJ431

Commit message: g
Parts:
- removed C32, C33: 1u, Capacitor_SMD:C_0402_1005Metric, symbol Device:C_Small
- removed C8: 100n, Capacitor_SMD:C_0603_1608Metric, symbol Device:C
- removed D2, D3, D4, D5: green, LED_SMD:LED_0805_2012Metric, symbol Device:LED_Small
- removed J1, J6: Conn_01x04, Connector_PinHeader_2.54mm:PinHeader_1x04_P2.54mm_Vertical, symbol Connector_Generic:Conn_01x04
- removed J3: Conn_01x06, Connector_PinHeader_2.54mm:PinHeader_1x06_P2.54mm_Vertical, symbol Connector_Generic:Conn_01x06
- removed J4: pins, Connector_PinHeader_2.54mm:PinHeader_1x02_P2.54mm_Vertical, symbol Connector_Generic:Conn_01x02
- removed R18: DNF, Resistor_SMD:R_0603_1608Metric_Pad0.98x0.95mm_HandSolder, symbol Device:R
- removed R19: 1k, Resistor_SMD:R_0603_1608Metric, symbol Device:R
- removed R27, R38, R66, R71: 10k, Resistor_SMD:R_0603_1608Metric, symbol Device:R_Small
- removed R28, R29, R30, R31: 1k, Resistor_SMD:R_0805_2012Metric, symbol Device:R
- removed SW2: MCU_RESET, SamacSys_Parts:PTS526SK15SMTR2LFS, symbol Switch:SW_SPST
- removed U10: MCP6002-xSN, Package_SO:SOIC-8_3.9x4.9mm_P1.27mm, symbol Amplifier_Operational:MCP6002-xSN
- removed U5: W25Q128JVS, Package_SO:SOIC-8_5.23x5.23mm_P1.27mm, symbol Memory_Flash:W25Q128JVS
- added C13: 1u, Capacitor_SMD:C_0402_1005Metric, symbol Device:C_Small
- added Q20, Q21: MMBT5551L, Package_TO_SOT_SMD:SOT-23, symbol Transistor_BJT:MMBT5551L
- added R34 (x2): 10k, Resistor_SMD:R_0603_1608Metric, symbol Device:R_Small
- added U13: MCP6002-xSN, Package_SO:SOIC-8_3.9x4.9mm_P1.27mm, symbol Amplifier_Operational:MCP6002-xSN
Connections:
- net CLK_EXT is gone; now on an unnamed net: J2.3 (Pin_3)
- net SCLK is gone; now on net BEMC_Phase_A: U1.9 (GPIO16/U0CTS/ADC2_CH5/XTAL_32K_N)
- net SS_EXT is gone; now on an unnamed net: J2.2 (Pin_2)
- net +3V3: now also J2.6 (Pin_6), C13.2, U13.8 (V+); no longer J2.1 (Pin_1)
- net 2V5_RAW: now also U13.5 (+)
- net BEMC_Phase_A_2: now also U1.35 (MTMS/GPIO42)
- net BEMC_Phase_B: now also U1.20 (GPIO12/TOUCH12/ADC2_CH1/FSPICLK/FSPIIO6/SUBSPICLK)
- net BEMC_Phase_B_2: now also U1.22 (GPIO14/TOUCH14/ADC2_CH3/FSPIWP/FSPIDQS/SUBSPIWP)
- net BEMC_Phase_C: now also U1.10 (GPIO17/U1TXD/ADC2_CH6)
- net BEMC_Phase_C_2: now also U1.23 (GPIO21)
- net Current_Out1: now also U1.12 (GPIO8/TOUCH8/ADC1_CH7/SUBSPICS1)
- net Current_Out2: now also U1.19 (GPIO11/TOUCH11/ADC2_CH0/FSPID/FSPIIO5/SUBSPID)
- net ESP_BOOT: now also SW3.2 (B), Q21.3 (C); no longer SW3.1 (A)
- net ESP_EN: now also Q20.3 (C)
- net GND: now also J2.1 (Pin_1), SW3.1 (A), C13.1, U13.4 (V-); no longer J2.6 (Pin_6), SW3.2 (B)
- net Phase_A_H: now also U1.11 (GPIO18/U1RXD/ADC2_CH7/CLK_OUT3)
- net Phase_A_H_2: now also U1.32 (MTCK/GPIO39/CLK_OUT3/SUBSPICS1)
- net Phase_A_L: now also U1.21 (GPIO13/TOUCH13/ADC2_CH2/FSPIQ/FSPIIO7/SUBSPIQ)
- net Phase_A_L_2: now also U1.28 (SPIIO6/GPIO35/FSPID/SUBSPID)
- net Phase_B_H: now also U1.4 (GPIO4/TOUCH4/ADC1_CH3)
- net Phase_B_H_2: now also U1.30 (SPIDQS/GPIO37/FSPIQ/SUBSPIQ)
- net Phase_B_L: now also U1.5 (GPIO5/TOUCH5/ADC1_CH4)
- net Phase_B_L_2: now also U1.33 (MTDO/GPIO40/CLK_OUT2)
- net Phase_C_H: now also U1.6 (GPIO6/TOUCH6/ADC1_CH5)
- net Phase_C_H_2: now also U1.29 (SPIIO7/GPIO36/FSPICLK/SUBSPICLK)
- net Phase_C_L: now also U1.7 (GPIO7/TOUCH7/ADC1_CH6)
- net Phase_C_L_2: now also U1.34 (MTDI/GPIO41/CLK_OUT1)
- net REF_2v5: now also U1.18 (GPIO10/TOUCH10/ADC1_CH9/FSPICS0/FSPIIO4/SUBSPICS0), U13.6 (-), U13.7
- net current: now reaches U1.17 (GPIO9/TOUCH9/ADC1_CH8/FSPIHD/SUBSPIHD)
- net GPIO_47: now reaches U1.24 (GPIO47/SPICLK_P/SUBSPICLK_P_DIFF)
- net GPIO_48: now reaches U1.25 (GPIO48/SPICLK_N/SUBSPICLK_N_DIFF)
- net GPIO_38: now reaches U1.31 (GPIO38/FSPIWP/SUBSPIWP)
- net GPIO_02: now reaches U1.38 (GPIO2/TOUCH2/ADC1_CH1)
- net GPIO_01: now reaches U1.39 (GPIO1/TOUCH1/ADC1_CH0)
- net +BATT renamed VDC
- net MISO renamed GPIO_15
- net MISO_EXT renamed DTR
- net DTR: now also Q21.2 (E), R34.1
- net MOSI_EXT renamed RST
- net RST: now also Q20.2 (E), R34.1
- new net: Q21.1 (B), R34.2
- new net: Q20.1 (B), R34.2
Other:
- note removed: "5ms delay or more"
- note removed: "Flash"
- note removed: "INMP441"
- note removed: "Max memory: 128Mbit chip (16Mbyte) must be : quad SPI flash memory"
- moved on the sheet: C13, C14, C15, C31, C34, C37, C57, D6, D7, D8, FB1, FID1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

Commit message: l
Connections:
- net GPIO_01 is gone; now on net SDA: U1.39 (GPIO1/TOUCH1/ADC1_CH0)
- net GPIO_02 is gone; now on net SCL: U1.38 (GPIO2/TOUCH2/ADC1_CH1)
- net RX: now reaches J2.2 (Pin_2), U1.37 (U0TXD/GPIO43/CLK_OUT1)
- net TX: now reaches J2.3 (Pin_3), U1.36 (U0RXD/GPIO44/CLK_OUT2)
Changed lines of the file:
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@@
+    (stroke (width 0) (type default))
+  )
+  (wire (pts (xy 331.47 246.38) (xy 314.96 246.38))
     (stroke (width 0) (type default))
   )
@@
   )
   (wire (pts (xy 68.58 163.83) (xy 66.04 163.83))
+    (stroke (width 0) (type default))
+  )
+  (wire (pts (xy 331.47 248.92) (xy 314.96 248.92))
     (stroke (width 0) (type default))
   )
@@
     (effects (font (size 1.27 1.27)) (justify left bottom))
   )
-  (label "GPIO_48" (at 354.33 127 0) (fields_autoplaced)
+  (label "GPIO_01" (at 314.96 248.92 0) (fields_autoplaced)
     (effects (font (size 1.27 1.27)) (justify left bottom))
   )
@@
     (effects (font (size 1.27 1.27)) (justify right bottom))
   )
-  (label "GPIO_38" (at 354.33 119.38 0) (fields_autoplaced)
+  (label "RX" (at 208.28 50.8 0) (fields_autoplaced)
     (effects (font (size 1.27 1.27)) (justify left bottom))
   )
@@
     (effects (font (size 1.27 1.27)) (justify left bottom))
   )
+  (label "GPIO_02" (at 314.96 246.38 0) (fields_autoplaced)
+    (effects (font (size 1.27 1.27)) (justify left bottom))
+  )
   (label "GPIO_07" (at 208.28 87.63 0) (fields_autoplaced)
     (effects (font (size 1.27 1.27)) (justify left bottom))
@@
     (effects (font (size 1.27 1.27)) (justify left bottom))
   )
+  (label "TX" (at 208.28 48.26 0) (fields_autoplaced)
+    (effects (font (size 1.27 1.27)) (justify left bottom))
+  )
   (label "GPIO_37" (at 314.96 207.01 0) (fields_autoplaced)
     (effects (font (size 1.27 1.27)) (justify left bottom))
@@
     (effects (font (size 1.27 1.27)) (justify right bottom))
   )
-  (label "GPIO_15" (at 354.33 121.92 0) (fields_autoplaced)
-    (effects (font (size 1.27 1.27)) (justify left bottom))
-  )
   (label "GPIO_18" (at 314.96 171.45 0) (fields_autoplaced)
     (effects (font (size 1.27 1.27)) (justify left bottom))
@@
     (effects (font (size 1.27 1.27)) (justify left bottom))
   )
-  (label "GPIO_47" (at 354.33 124.46 0) (fields_autoplaced)
-    (effects (font (size 1.27 1.27)) (justify left bottom))
-  )
   (global_label "SDA" (shape input) (at 208.28 265.43 180) (fields_autoplaced)
     (effects (font (size 1.27 1.27)) (justify right))
@@
     (property "Intersheetrefs" "${INTERSHEET_REFS}" (at 77.2945 203.2794 0)
       (effects (font (size 1.27 1.27)) (justify right) hide)
+    )
+  )
+  (global_label "SCL" (shape input) (at 331.47 246.38 0) (fields_autoplaced)
+    (effects (font (size 1.27 1.27)) (justify left))
+    (property "Intersheetrefs" "${INTERSHEET_REFS}" (at 337.8834 246.38 0)
+      (effects (font (size 1.27 1.27)) (justify left) hide)
     )
   )
@@
       (effects (font (size 1.27 1.27)) (justify left) hide)
     )
+  )
+  (global_label "SDA" (shape input) (at 331.47 248.92 0) (fields_autoplaced)
+    (effects (font (size 1.27 1.27)) (justify left))
+    (property "Intersheetrefs" "${INTERSHEET_REFS}" (at 337.9439 248.92 0)
+      (effects (font (size 1.27 1.27)) (justify left) hide)
+    )

Commit message: g
Parts:
- removed C37: 1n, Capacitor_SMD:C_1206_3216Metric, symbol Device:C_Small
- removed J4: USB_C_Receptacle, Connector_USB:USB_C_Receptacle_HRO_TYPE-C-31-M-12, symbol Connector:USB_C_Receptacle
- removed R32, R33: 5k1, Resistor_SMD:R_0402_1005Metric, symbol Device:R_Small
- added J2: USB_A, Connector_USB:USB_A_Molex_67643_Horizontal, symbol Connector:USB_A
- added RV1, RV2: R_Potentiometer_MountingPin, Potentiometer_THT:Potentiometer_Alps_RK09K_Single_Vertical, symbol Device:R_Potentiometer_MountingPin
Connections:
- net GPIO_38 is gone; now on net BEMC_Phase_A: U1.31 (GPIO38/FSPIWP/SUBSPIWP)
- net +3V3: now also RV1.3, RV2.3
- net BEMC_Phase_A: no longer U1.9 (GPIO16/U0CTS/ADC2_CH5/XTAL_32K_N)
- net D+: now also J2.3 (D+)
- net D-: now also J2.2 (D-)
- net GND: now also J2.4 (GND), RV1.1, RV1.MP (MountPin), RV2.1, RV2.MP (MountPin)
- net GPIO_15: now also RV2.2
- net VBUS: now also J2.1 (VBUS)
- new net GPIO_16: RV1.2, U1.9 (GPIO16/U0CTS/ADC2_CH5/XTAL_32K_N)
- no-connect marks 19 -> 10
