File: ESP32_dual_ESC/POWER.kicad_sch (KiCad schematic)
At the start: 7 parts, among them Q1 N MOSFET, U12 INA219AxD

Commit message: g
Parts:
- removed Q1: N MOSFET, Package_DFN_QFN:PQFN-8-EP_6x5mm_P1.27mm_Generic, symbol Device:Q_NMOS_DSG
- added J1 (x2): A, MountingHole:MountingHole_2.5mm_Pad_TopBottom, symbol Connector_Generic:Conn_01x01
- added R15 (x2): 1k, Resistor_SMD:R_0402_1005Metric, symbol Device:R_Small
- added R6 (x2): 75k, Resistor_SMD:R_0402_1005Metric, symbol Device:R_Small
- added U13: MCP6002-xSN, Package_SO:SOIC-8_3.9x4.9mm_P1.27mm, symbol Amplifier_Operational:MCP6002-xSN
Connections:
- net GND: now also U12.1 (A1), U12.2 (A0), J1.1 (Pin_1), R6.1
- net VDC: now also J1.1 (Pin_1), R15.1
- net VCC renamed +15V
- net +15V: now also R15.1
- new net: R15.2, R6.1, U13.3 (+)
- new net: R15.2, R6.2, U13.2 (-)
- new net current: R6.2, U13.1
Other:
- moved on the sheet: C15, C25, R56, R57, R58, U12

Commit message: l
Parts:
- added C13 (x2): 1u, Capacitor_SMD:C_0402_1005Metric, symbol Device:C_Small
- added C14 (x2): 10u, Capacitor_SMD:C_0603_1608Metric, symbol Device:C_Small
- added C23: 100u, Capacitor_SMD:CP_Elec_6.3x5.4, symbol Device:C_Polarized_US
- added C8: 100n, Capacitor_SMD:C_0603_1608Metric, symbol Device:C_Small
- added D1 (x3): B5819W_SL, Diode_SMD:D_SOD-123, symbol Device:D_Small
- added D6: green, LED_SMD:LED_0805_2012Metric, symbol Device:LED_Small
- added J4: Conn_01x02, Connector_PinHeader_2.54mm:PinHeader_1x02_P2.54mm_Vertical, symbol Connector_Generic:Conn_01x02
- added JP1: Jumper_2_Bridged, Jumper:SolderJumper-2_P1.3mm_Bridged_RoundedPad1.0x1.5mm, symbol Jumper:Jumper_2_Bridged
- added L1: 75u, Inductor_SMD:L_Changjiang_FNR8040S, symbol Device:L
- added R15 (x2): 10K, Resistor_SMD:R_0603_1608Metric, symbol Device:R_Small
- added R68: 6.2k, Resistor_SMD:R_0603_1608Metric, symbol Device:R
- added U5: TPS5430DDA, Package_SO:TI_SO-PowerPAD-8_ThermalVias, symbol Regulator_Switching:TPS5430DDA
Connections:
- net +15V: now also D1.2 (A), D6.2 (A)
- net +3V3: now also C13.2, C14.1, C23.1, L1.1, R15.2
- net GND: now also C13.1, C13.1, C14.2, C14.2, C23.2, D1.2 (A), J4.1 (Pin_1), JP1.1 (A), R68.2, U5.6 (GND), U5.9 (GNDPAD)
- new net: C13.2, C14.1, D1.1 (K), D1.1 (K), U5.7 (VIN)
- new net: J4.2 (Pin_2), U5.5 (EN)
- new net: C8.1, D1.1 (K), L1.2, U5.8 (PH)
- new net: C8.2, U5.1 (BOOT)
- new net: JP1.2 (B), R15.1
- new net: D6.1 (K), R15.2
- new net: R15.1, R68.1, U5.4 (VSENSE)
- new net +5V: D1.2 (A)

Commit message: g
Parts:
- added C14 (x2): 10u, Capacitor_SMD:C_0603_1608Metric, symbol Device:C_Small
- added R13: 2k, Resistor_SMD:R_0402_1005Metric, symbol Device:R_Small
- added R13: 470, Resistor_SMD:R_0402_1005Metric, symbol Device:R_Small
- added R34 (x2): 10k, Resistor_SMD:R_0603_1608Metric, symbol Device:R_Small
- added U8: LM317_TO-220, Package_TO_SOT_THT:TO-220-3_Vertical, symbol Regulator_Linear:LM317_TO-220
Connections:
- net +15V: now also C14.1, R13.1, U8.2 (VO); no longer D1.2 (A), D6.2 (A), R15.1, R56.1, R57.1
- net GND: now also C14.2, C14.2, R34.1
- new net: R34.1, R34.2
- new net: R13.2, R13.2
- new net: R13.1, R34.2, U8.1 (ADJ)
- new net VCC: C14.1, D1.2 (A), D6.2 (A), R15.1, R56.1, R57.1, U8.3 (VI)
Other:
- moved on the sheet: C13, C14, C23, C8, D1, J4, L1, R15, R68, U5
