File: ESP32_dual_ESC/_autosave-ESP32_dual_ESC.kicad_pcb (KiCad board)
At the start: 4 copper layers, 100 x 100 mm, 193 parts, among them J1 A, J10 Conn_01x04, J11 A, J12 B, J13 C, J14 A, J15 A, J2 B, J3 C, J4 Conn_01x02, J5 USB_A, J7 Conn_01x06, Q1 HYG025N06LS1C2, Q10 HYG025N06LS1C2, Q11 HYG025N06LS1C2, Q12 HYG025N06LS1C2, Q2 HYG025N06LS1C2, Q20 MMBT5551L, Q21 MMBT5551L, Q3 HYG025N06LS1C2, Q4 HYG025N06LS1C2, Q5 HYG025N06LS1C2, Q6 HYG025N06LS1C2, Q7 HYG025N06LS1C2, Q8 HYG025N06LS1C2, Q9 HYG025N06LS1C2, SW1 MCU_RESET, SW3 MCU_RESET, U1 LM324, U10 LM324, U11 DRV8300N, U12 INA219AxD, U13 MCP6002-xSN, U2 LM5109BMA, U3 LM5109BMA, U4 LM5109BMA, U5 TPS5430DDA, U6 ESP32-S3-WROOM-1, U7 SRV05-4, U8 LM317_TO-220, U9 CJ431

Commit message: g
Parts:
- moved FID3 7.32 mm to (144.8, 135.1)
Changed lines of the file:
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@@
     (property "Sheetname" "MCU")
     (attr smd)
-    (fp_text reference "U9" (at -1.1775 2.79 180) (layer "F.SilkS")
+    (fp_text reference "U9" (at 2.6625 0.98 180) (layer "F.SilkS")
         (effects (font (size 1 1) (thickness 0.15)))
     )
@@
     (property "ki_keywords" "resistor variable")
     (attr through_hole)
-    (fp_text reference "RV2" (at 6.05 -5.15 90) (layer "F.SilkS")
+    (fp_text reference "RV2" (at -2.07 2.64) (layer "F.SilkS")
         (effects (font (size 1 1) (thickness 0.15)))
     )
@@
     (property "ki_keywords" "resistor variable")
     (attr through_hole)
-    (fp_text reference "RV1" (at 6.05 -5.15 90) (layer "F.SilkS")
+    (fp_text reference "RV1" (at -2.01 2.57) (layer "F.SilkS")
         (effects (font (size 1 1) (thickness 0.15)))
     )
@@
   )
   (footprint "Symbol:WEEE-Logo_4.2x6mm_SilkScreen" (layer "F.Cu")
-    (at 138 132.44)
+    (at 144.83 135.07)
     (descr "Waste Electrical and Electronic Equipment Directive")
     (tags "Logo WEEE")
@@
   (via (at 129.41 103.34) (size 0.7) (drill 0.4) (layers "F.Cu" "B.Cu") (free) (net 1))
   (via (at 96.44 141.05) (size 0.65) (drill 0.35) (layers "F.Cu" "B.Cu") (net 1))
-  (via (at 88.354 59.576) (size 3) (drill 2.5) (layers "F.Cu" "B.Cu") (free) (net 1))
+  (via (at 88.53 59.48) (size 3) (drill 2.5) (layers "F.Cu" "B.Cu") (free) (net 1))
   (via (at 80.545382 72.611797) (size 0.7) (drill 0.4) (layers "F.Cu" "B.Cu") (free) (net 1))
   (via (at 108.46 103.15) (size 0.7) (drill 0.4) (layers "F.Cu" "B.Cu") (net 1))
