File: ESP32_dual_ESC_v2/ESC_V1.kicad_sch (KiCad schematic)
At the start: 58 parts, among them J1 A, J2 B, J3 C, Q1 HYG025N06LS1C2, Q2 HYG025N06LS1C2, Q3 HYG025N06LS1C2, Q4 HYG025N06LS1C2, Q5 HYG025N06LS1C2, Q6 HYG025N06LS1C2, U1 LM324, U2 LM5109BMA, U3 LM5109BMA, U4 LM5109BMA

Commit message: 3
Parts:
- U1: footprint (none) -> Package_SO:SOIC-14_3.9x8.7mm_P1.27mm
- renumbered C31 to C7, D7 to D16, D15 to D17, D7 to D18, D15 to D19, D7 to D20, D15 to D21, R56 to R3
Connections:
- net ESC1_VCC renamed ESC_VCC
