File: ESP32_dual_ESC_v2/ESC_V2.kicad_sch (KiCad schematic)
At the start: 55 parts, among them J1 A, J2 B, J3 C, Q1 HYG025N06LS1C2, Q2 HYG025N06LS1C2, Q3 HYG025N06LS1C2, Q4 HYG025N06LS1C2, Q5 HYG025N06LS1C2, Q6 HYG025N06LS1C2, U1 LM324, U11 DRV8300N

Commit message: 3
Parts:
- renumbered C2 to C15, C2 to C16, C2 to C19, C2 to C20, C2 to C22, C2 to C66, C2 to C67, C2 to C68, C2 to C69, C2 to C70, C2 to C71, D1 to D11, D2 to D12, D3 to D13, J1 to J11, J2 to J12, J3 to J13, Q4 to Q10, Q5 to Q11, Q6 to Q12, Q1 to Q7, Q2 to Q8, Q3 to Q9, R15 to R25, R15 to R26, R16 to R28, R16 to R29, R16 to R30, R16 to R31, R16 to R37, R16 to R39, R6 to R40, R56 to R41, R5 to R43, R6 to R44, R7 to R45, R8 to R46, R9 to R47, R9 to R48, R9 to R49, R12 to R50, R13 to R51, R14 to R52, R15 to R53, R16 to R54, R17 to R55, U1 to U10
