File: ESP32_dual_ESC_v2/POWER.kicad_sch (KiCad schematic)
At the start: 37 parts, among them J1 A, J4 Conn_01x02, U12 INA219AxD, U13 MCP6002-xSN, U5 TPS5430DDA, U8 LM317_TO-220

Commit message: 3
Parts:
- added C44, C46: 1u, Capacitor_SMD:C_0402_1005Metric, symbol Device:C_Small
- added C45, C47: 10u, Capacitor_SMD:C_0603_1608Metric, symbol Device:C_Small
- added D26: B5819W_SL, Diode_SMD:D_SOD-123, symbol Device:D_Small
- added U20: LM1117T-3.3, Package_TO_SOT_THT:TO-220-3_Vertical, symbol Regulator_Linear:LM1117T-3.3
- renumbered D1 to D22, D1 to D23, D1 to D24, J1 to J14, J1 to J15, R15 to R27, R15 to R64, R6 to R65, R15 to R66, R6 to R67, R15 to R69
Connections:
- net +3V3: now also C44.2, C45.1, U20.2 (VO)
- net GND: now also C44.1, C45.2, C46.1, C47.2, U20.1 (GND)
- net at C13.2, C14.1, D22.1 (K)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: now also C46.2, C47.1, D26.1 (K), U20.3 (VI)
- new net 5v_2: D26.2 (A)

Commit message: 6
Parts:
- U20: footprint Package_TO_SOT_THT:TO-220-3_Vertical -> Package_TO_SOT_THT:TO-220-3_Horizontal_TabDown; now fitted
- U8: footprint Package_TO_SOT_THT:TO-220-3_Vertical -> Package_TO_SOT_THT:TO-220-3_Horizontal_TabDown
Changed lines of the file:
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@@
 		(in_bom yes)
 		(on_board yes)
-		(dnp yes)
+		(dnp no)
 		(fields_autoplaced yes)
 		(property "Reference" "U20"
@@
 			)
 		)
-		(property "Footprint" "Package_TO_SOT_THT:TO-220-3_Vertical"
+		(property "Footprint" "Package_TO_SOT_THT:TO-220-3_Horizontal_TabDown"
 			(at 246.38 95.25 0)
 			(effects
@@
 			)
 		)
-		(property "Footprint" "Package_TO_SOT_THT:TO-220-3_Vertical"
+		(property "Footprint" "Package_TO_SOT_THT:TO-220-3_Horizontal_TabDown"
 			(at 177.8 23.495 0)
 			(effects
