File: ESP32_dual_ESC_v2/ESP32_dual_ESC.kicad_pcb (KiCad board)
At the start: 4 copper layers, 100 x 100 mm, 245 parts, among them J1 A, J10 Conn_01x04, J14 A, J15 A, J2 B, J3 C, J4 Conn_01x02, J5 USB_A, J6 USB_A, J7 C, J8 B, J9 A, Q1 HYG025N06LS1C2, Q10 HYG025N06LS1C2, Q11 HYG025N06LS1C2, Q12 HYG025N06LS1C2, Q2 HYG025N06LS1C2, Q20 MMBT5551L, Q21 MMBT5551L, Q3 HYG025N06LS1C2, Q4 HYG025N06LS1C2, Q5 HYG025N06LS1C2, Q6 HYG025N06LS1C2, Q7 HYG025N06LS1C2, Q8 HYG025N06LS1C2, Q9 HYG025N06LS1C2, SW1 MCU_RESET, SW3 MCU_RESET, U1 LM324, U10 LM324, U11 LM5109BMA, U12 INA219AxD, U13 MCP6002-xSN, U14 SRV05-4, U15 CP2102N-Axx-xQFN28, U16 SN74AVC8T245PW, U17 LM5109BMA, U18 LM5109BMA, U19 MCP6002-xSN, U2 LM5109BMA, U20 LM1117T-3.3, U3 LM5109BMA, U4 LM5109BMA, U5 TPS5430DDA, U6 ESP32-S3-WROOM-1, U7 SRV05-4, U8 LM317_TO-220, U9 CJ431

Commit message: 6
Parts:
- J6: moved to B.Cu
- U20, U8: footprint Package_TO_SOT_THT:TO-220-3_Vertical -> Package_TO_SOT_THT:TO-220-3_Horizontal_TabDown
- moved C7 167.7 mm to (91.9, 116.7)
- moved C42 104.0 mm to (104.3, 80.9), turned to 90 degrees
- moved C43 102.9 mm to (105.3, 73.0), turned to -90 degrees
- moved C46 98.6 mm to (125.2, 80.2), turned to 90 degrees
- moved C47 95.6 mm to (126.5, 80.2), turned to -90 degrees
- moved C44 95.2 mm to (125.2, 83.6), turned to 90 degrees
- moved FB2 94.7 mm to (120.3, 55.8)
- moved R90 92.0 mm to (105.3, 82.4)
- moved C45 91.7 mm to (126.5, 83.6), turned to -90 degrees
- moved R39 89.5 mm to (107.5, 118.5)
- moved R43 89.0 mm to (109.4, 117.3), turned to 180 degrees
- moved R29 88.6 mm to (107.5, 117.3), turned to 180 degrees
- moved R30 87.0 mm to (109.4, 118.5)
- moved JP2 70.7 mm to (93.7, 83.7), turned to 180 degrees
- moved R69 68.2 mm to (93.6, 86.0), turned to 0 degrees
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Routing:
- net SCL: track 29.2 -> 126.2 mm, vias 2 -> 1
- net SDA: track 27.5 -> 123.9 mm, vias 2 -> 1
- net VCC: track 28.8 -> 99.9 mm
- net +15V: track 51.6 -> 120.4 mm, vias 1 -> 2
- net Net-(D22-K): track 14.3 -> 64.3 mm
- net /ESC_V2/Phase_A_H: track 0.00 -> 39.5 mm
- net /ESC_V2/Phase_A_L: track 0.00 -> 38.3 mm, vias 0 -> 1
- net /ESC_V1/Phase_A_H: track 0.00 -> 37.8 mm
- net 5v_2: track 0.00 -> 34.7 mm
- net /ESC_V1/Phase_A_L: track 0.00 -> 34.2 mm
- net /MCU/ESP_EN: track 38.6 -> 71.4 mm, vias 2 -> 3
- net /ESC_V2/Phase_B_L: track 0.00 -> 28.2 mm
- net /ESC_V2/Phase_B_H: track 0.00 -> 28.0 mm
- net /ESC_V1/Phase_B_H: track 0.00 -> 25.8 mm
- net +5V: track 25.1 -> 47.5 mm, vias 2 -> 3
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- removed copper zone on F.Cu, net Net-(U10A-+)

Commit message: tg
Parts:
- added TP8: TestPoint, TestPoint:TestPoint_Pad_1.0x1.0mm, F.Cu at (92.7, 73.5)
- added TP9: TestPoint, TestPoint:TestPoint_Pad_1.0x1.0mm, F.Cu at (95.8, 73.5)
- moved R93 48.9 mm to (74.7, 131.5), turned to 90 degrees
- moved R94 20.0 mm to (132.9, 131.3), turned to 90 degrees
- moved R19 5.25 mm to (108.8, 63.3), turned to 90 degrees
- moved R18 4.83 mm to (112.7, 60.1), turned to -90 degrees
- moved Q20 4.17 mm to (111.4, 63.8), turned to -90 degrees
- moved Q21 3.95 mm to (110.0, 60.0), turned to 180 degrees
- moved FB2 3.15 mm to (117.3, 56.6)
Connections:
- net Net-(U6-U0RXD/GPIO44/CLK_OUT2) renamed /MCU/TX_in
- net Net-(U6-U0TXD/GPIO43/CLK_OUT1) renamed /MCU/RX_in
- R83 pad 2: /MCU/GPIO_39 -> /MCU/GPIO_35
- R84 pad 2: /MCU/GPIO_35 -> /MCU/GPIO_37
- R85 pad 2: /MCU/GPIO_37 -> /MCU/GPIO_39
- U11 pad 2: /MCU/GPIO_36 -> /ESC_V2/Phase_C_H
- U16 pad 4: /ESC_V2/Phase_A_L -> /ESC_V2/Phase_B_L
- U16 pad 6: /ESC_V2/Phase_B_L -> /ESC_V2/Phase_C_L
- U16 pad 7: /ESC_V2/Phase_C_L -> /ESC_V2/Phase_C_H
- U18 pad 3: /ESC_V2/Phase_A_L -> /MCU/GPIO_36
Routing:
- net /MCU/GPIO_36: track 14.8 -> 60.8 mm, vias 0 -> 2
- net /MCU/TX_in: track 0.00 -> 40.1 mm
- net /ESC_V2/Phase_A_L: track 38.3 -> 0.00 mm, vias 1 -> 0
- net /MCU/RX_in: track 0.00 -> 37.9 mm
- net /MCU/GPIO_05: track 0.00 -> 26.5 mm, vias 0 -> 2
- net /MCU/GPIO_04: track 0.00 -> 26.0 mm, vias 0 -> 2
- net /MCU/GPIO_06: track 0.00 -> 25.0 mm, vias 0 -> 2
- net /ESC_V2/A1: track 18.9 -> 43.3 mm, vias 52 -> 54
- net /MCU/GPIO_38: track 0.00 -> 23.0 mm, vias 0 -> 2
- net /MCU/GPIO_17: track 0.00 -> 22.1 mm, vias 0 -> 2
- net /MCU/GPIO_07: track 0.00 -> 21.6 mm, vias 0 -> 2
- net /MCU/GPIO_18: track 0.00 -> 19.8 mm, vias 0 -> 2
- net /MCU/GPIO_40: track 0.00 -> 17.9 mm
- net +15V: track 120.4 -> 103.0 mm
- net /MCU/GPIO_41: track 0.00 -> 17.2 mm
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