File: ESP32_dual_ESC_v2/MCU.kicad_sch (KiCad schematic)
At the start: 44 parts, among them J2 Conn_01x06, J2 USB_A, J5 Conn_01x04, Q20 MMBT5551L, Q21 MMBT5551L, SW1 MCU_RESET, SW3 MCU_RESET, U1 ESP32-S3-WROOM-1, U13 MCP6002-xSN, U4 SRV05-4, U9 CJ431

Commit message: 3
Parts:
- removed J2: Conn_01x06, Connector_PinHeader_2.54mm:PinHeader_1x06_P2.54mm_Vertical, symbol Connector_Generic:Conn_01x06
- added C13 (x2), C41, C42, C43: 1u, Capacitor_SMD:C_0402_1005Metric, symbol Device:C_Small
- added C14: 10u, Capacitor_SMD:C_0603_1608Metric, symbol Device:C_Small
- added FB1: FerriteBead_Small, Resistor_SMD:R_0805_2012Metric, symbol Device:FerriteBead_Small
- added J2: USB_A, Connector_USB:USB_A_Molex_67643_Horizontal, symbol Connector:USB_A
- added R34, R72, R91, R93, R94: 10k, Resistor_SMD:R_0603_1608Metric, symbol Device:R_Small
- added R73, R74, R75, R76, R77, R78, R79, R80, R81, R83, R84, R85, R86, R87, R88, R89, R90, R95, R96, R97: 0, Resistor_SMD:R_0402_1005Metric_Pad0.72x0.64mm_HandSolder, symbol Device:R_Small
- added R92: 2k, Resistor_SMD:R_0402_1005Metric, symbol Device:R_Small
- added TP2, TP3, TP4, TP5, TP6, TP7: TestPoint, TestPoint:TestPoint_Pad_1.0x1.0mm, symbol Connector:TestPoint
- added U15: CP2102N-Axx-xQFN28, Package_DFN_QFN:QFN-28-1EP_5x5mm_P0.5mm_EP3.35x3.35mm, symbol Interface_USB:CP2102N-Axx-xQFN28
- added U16: SN74AVC8T245PW, Package_SO:TSSOP-24_4.4x7.8mm_P0.65mm, symbol Logic_LevelTranslator:SN74AVC8T245PW
- added U19: MCP6002-xSN, Package_SO:SOIC-8_3.9x4.9mm_P1.27mm, symbol Amplifier_Operational:MCP6002-xSN
- added U4: SRV05-4, Package_TO_SOT_SMD:SOT-23-6, symbol Power_Protection:SRV05-4
Connections:
- net +3V3: now also C41.2, C42.2, R72.2, U16.1 (VCCA), U19.8 (V+); no longer RV1.3, RV2.3
- net BEMC_Phase_A: now also R79.1; no longer U1.31 (GPIO38/FSPIWP/SUBSPIWP)
- net BEMC_Phase_B: now also R80.1; no longer U1.20 (GPIO12/TOUCH12/ADC2_CH1/FSPICLK/FSPIIO6/SUBSPICLK)
- net BEMC_Phase_C: now also R81.1; no longer U1.10 (GPIO17/U1TXD/ADC2_CH6)
- net DTR: now also U15.28 (~{DTR})
- net GND: now also C13.1, C13.1, C14.2, C41.1, C42.1, C43.1, J2.4 (GND), R89.2, R90.1, R92.2, R95.1, U15.29 (GND), U15.3 (GND), U16.11 (GND), U16.12 (GND), U16.13 (GND), U19.4 (V-), U4.2 (VN)
- net Phase_A_H: now also R73.1; no longer U1.11 (GPIO18/U1RXD/ADC2_CH7/CLK_OUT3)
- net Phase_A_H_2: now also U16.3 (A1); no longer U1.32 (MTCK/GPIO39/CLK_OUT3/SUBSPICS1)
- net Phase_A_L: now also R74.1; no longer U1.21 (GPIO13/TOUCH13/ADC2_CH2/FSPIQ/FSPIIO7/SUBSPIQ)
- net Phase_A_L_2: now also U16.4 (A2); no longer U1.28 (SPIIO6/GPIO35/FSPID/SUBSPID)
- net Phase_B_H: now also R75.1; no longer U1.4 (GPIO4/TOUCH4/ADC1_CH3)
- net Phase_B_H_2: now also U16.5 (A3); no longer U1.30 (SPIDQS/GPIO37/FSPIQ/SUBSPIQ)
- net Phase_B_L: now also R76.1; no longer U1.5 (GPIO5/TOUCH5/ADC1_CH4)
- net Phase_B_L_2: now also U16.6 (A4); no longer U1.33 (MTDO/GPIO40/CLK_OUT2)
- net Phase_C_H: now also R77.1; no longer U1.6 (GPIO6/TOUCH6/ADC1_CH5)
- net Phase_C_L: now also R78.1; no longer U1.7 (GPIO7/TOUCH7/ADC1_CH6)
- net Phase_C_L_2: now also U16.7 (A5); no longer U1.34 (MTDI/GPIO41/CLK_OUT1)
- net RST: now also U15.24 (~{RTS})
- net RX: now also R96.2, U15.25 (RXD); no longer U1.37 (U0TXD/GPIO43/CLK_OUT1)
- net TX: now also R97.2, U15.26 (TXD); no longer U1.36 (U0RXD/GPIO44/CLK_OUT2)
- new net: R72.1, R91.2, U19.3 (+)
- new net: TP3.1, U16.15 (B7)
- new net: R90.2, U16.2 (DIR)
- new net: R34.1, U15.9 (~{RST})
- new net: C13.2, R34.2, U15.6 (VDD)
- new net: R94.1, RV2.3
- new net: R97.1, U1.36 (U0RXD/GPIO44/CLK_OUT2)
- new net: R88.2, TP2.1
- new net: R87.1, U16.17 (B5)
- new net: R96.1, U1.37 (U0TXD/GPIO43/CLK_OUT1)
- new net: R95.2, U19.5 (+)
- new net: R93.1, RV1.3
- new net: TP5.1, U16.8 (A6)
- new net: R91.1, R92.1
- new net: TP4.1, U16.14 (B8)
- new net: R83.1, U16.21 (B1)
- new net: R89.1, U16.22 (~{OE})
- new net: R88.1, U16.16 (B6)
- new net: TP7.1, U16.10 (A8)
- new net: R86.1, U16.18 (B4)
- new net: R85.1, U16.19 (B3)
- new net: R84.1, U16.20 (B2)
- new net: TP6.1, U16.9 (A7)
- new net: U19.6 (-), U19.7
- new net 1V8: C43.2, R93.2, R94.2, U16.23 (VCCB), U16.24 (VCCB), U19.1, U19.2 (-)
- new net 5v_2: FB1.1
- new net D2+: J2.3 (D+), U15.4 (D+), U4.1 (IO1)
- new net D2-: J2.2 (D-), U15.5 (D-), U4.6 (IO4)
- new net GPIO_04: R75.2, U1.4 (GPIO4/TOUCH4/ADC1_CH3)
- new net GPIO_05: R76.2, U1.5 (GPIO5/TOUCH5/ADC1_CH4)
- new net GPIO_06: R77.2, U1.6 (GPIO6/TOUCH6/ADC1_CH5)
- new net GPIO_07: R78.2, U1.7 (GPIO7/TOUCH7/ADC1_CH6)
- new net GPIO_12: R80.2, U1.20 (GPIO12/TOUCH12/ADC2_CH1/FSPICLK/FSPIIO6/SUBSPICLK)
- new net GPIO_13: R74.2, U1.21 (GPIO13/TOUCH13/ADC2_CH2/FSPIQ/FSPIIO7/SUBSPIQ)
- new net GPIO_17: R81.2, U1.10 (GPIO17/U1TXD/ADC2_CH6)
- new net GPIO_18: R73.2, U1.11 (GPIO18/U1RXD/ADC2_CH7/CLK_OUT3)
- new net GPIO_35: R84.2, U1.28 (SPIIO6/GPIO35/FSPID/SUBSPID)
- new net GPIO_37: R85.2, U1.30 (SPIDQS/GPIO37/FSPIQ/SUBSPIQ)
- new net GPIO_38: R79.2, U1.31 (GPIO38/FSPIWP/SUBSPIWP)
- new net GPIO_39: R83.2, U1.32 (MTCK/GPIO39/CLK_OUT3/SUBSPICS1)
- new net GPIO_40: R86.2, U1.33 (MTDO/GPIO40/CLK_OUT2)
- new net GPIO_41: R87.2, U1.34 (MTDI/GPIO41/CLK_OUT1)
- new net Vusb_2: C13.2, C14.1, FB1.2, J2.1 (VBUS), U15.7 (VREGIN), U15.8 (VBUS), U4.5 (VP)
- no-connect marks 10 -> 13
Other:
- moved on the sheet: Q20, Q21, R34, RV1, RV2

Commit message: tg
Parts:
- added TP8, TP9: TestPoint, TestPoint:TestPoint_Pad_1.0x1.0mm, symbol Connector:TestPoint
Connections:
- net GPIO_35: now also R83.2; no longer R84.2
- net GPIO_37: now also R84.2; no longer R85.2
- net GPIO_39: now also R85.2; no longer R83.2
- net GPIO_47: now also TP8.1
- net GPIO_48: now also TP9.1
- net Phase_A_L_2: now also U1.29 (SPIIO7/GPIO36/FSPICLK/SUBSPICLK); no longer U16.4 (A2)
- net Phase_B_L_2: now also U16.4 (A2); no longer U16.6 (A4)
- net Phase_C_H_2: now also U16.7 (A5); no longer U1.29 (SPIIO7/GPIO36/FSPICLK/SUBSPICLK)
- net Phase_C_L_2: now also U16.6 (A4); no longer U16.7 (A5)
- net TX_in: now reaches R97.1, U1.36 (U0RXD/GPIO44/CLK_OUT2)
- net RX_in: now reaches R96.1, U1.37 (U0TXD/GPIO43/CLK_OUT1)
Other:
- moved on the sheet: R96, R97
Changed lines of the file:
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@@
 	(wire
 		(pts
-			(xy 199.39 57.15) (xy 204.47 57.15)
+			(xy 191.77 57.15) (xy 198.12 57.15)
 		)
 		(stroke
@@
 	(wire
 		(pts
+			(xy 276.86 204.47) (xy 288.29 204.47)
+		)
+		(stroke
+			(width 0)
+			(type default)
+		)
+	)
+	(wire
+		(pts
 			(xy 269.24 240.03) (xy 285.75 240.03)
 		)
@@
 	(wire
 		(pts
-			(xy 218.44 54.61) (xy 215.9 54.61)
+			(xy 218.44 54.61) (xy 209.55 54.61)
 		)
 		(stroke
@@
 	(wire
 		(pts
+			(xy 276.86 207.01) (xy 288.29 207.01)
+		)
+		(stroke
+			(width 0)
+			(type default)
+		)
+	)
+	(wire
+		(pts
 			(xy 261.62 274.32) (xy 261.62 276.86)
 		)
@@
 	(wire
 		(pts
-			(xy 209.55 57.15) (xy 218.44 57.15)
+			(xy 203.2 57.15) (xy 218.44 57.15)
 		)
 		(stroke
@@
 	(wire
 		(pts
-			(xy 210.82 54.61) (xy 199.39 54.61)
+			(xy 204.47 54.61) (xy 191.77 54.61)
 		)
 		(stroke
@@
 	)
 	(label "RX"
-		(at 199.39 54.61 0)
+		(at 191.77 54.61 0)
 		(fields_autoplaced yes)
 		(effects
@@
 	)
 	(label "GPIO_35"
-		(at 327.66 226.06 0)
+		(at 327.66 223.52 0)
 		(fields_autoplaced yes)
 		(effects
@@
 		)
 	)
+	(label "TX_in"
+		(at 210.82 57.15 0)
+		(fields_autoplaced yes)
+		(effects
+			(font
+				(size 1.27 1.27)
+			)
+			(justify left bottom)
+		)
+	)
 	(label "GPIO_16"
 		(at 226.06 176.53 0)
@@
 	)
 	(label "GPIO_37"
-		(at 327.66 228.6 0)
+		(at 327.66 226.06 0)
 		(fields_autoplaced yes)
 		(effects
@@
 		)
 	)
+	(label "GPIO_48"
+		(at 276.86 207.01 0)
+		(fields_autoplaced yes)
+		(effects
+			(font
+				(size 1.27 1.27)
+			)
+			(justify left bottom)
+		)
+	)
+	(label "RX_in"
+		(at 210.82 54.61 0)
+		(fields_autoplaced yes)
+		(effects
+			(font
+				(size 1.27 1.27)
+			)
+			(justify left bottom)
+		)
+	)
 	(label "2V5_RAW"
 		(at 52.07 157.48 0)
@@
 	)
 	(label "GPIO_39"
-		(at 327.66 223.52 0)
+		(at 327.66 228.6 0)
 		(fields_autoplaced yes)
 		(effects
@@
 	)
 	(label "TX"
-		(at 199.39 57.15 0)
+		(at 191.77 57.15 0)
 		(fields_autoplaced yes)
 		(effects
@@
 		)
 	)
+	(label "GPIO_47"
+		(at 276.86 204.47 0)
+		(fields_autoplaced yes)
+		(effects
+			(font
+				(size 1.27 1.27)
+			)
+			(justify left bottom)
+		)
+	)
 	(label "GPIO_16"
 		(at 320.04 64.77 180)
@@
 	(hierarchical_label "Phase_A_L_2"
 		(shape input)
-		(at 383.54 226.06 0)
+		(at 285.75 229.87 0)
 		(fields_autoplaced yes)
 		(effects
@@
 	(hierarchical_label "Phase_B_L_2"
 		(shape input)
-		(at 383.54 231.14 0)
+		(at 383.54 226.06 0)
 		(fields_autoplaced yes)
 		(effects
@@
 	(hierarchical_label "Phase_C_H_2"
 		(shape input)
-		(at 285.75 229.87 0)
+		(at 383.54 233.68 0)
 		(fields_autoplaced yes)
 		(effects
@@
 	(hierarchical_label "Phase_C_L_2"
 		(shape input)
-		(at 383.54 233.68 0)
+		(at 383.54 231.14 0)
 		(fields_autoplaced yes)
 		(effects
@@
 	(symbol
 		(lib_id "Device:R_Small")
-		(at 207.01 57.15 270)
+		(at 200.66 57.15 270)
 		(mirror x)
 		(unit 1)
@@
 		(dnp no)
 		(property "Reference" "R97"
-			(at 204.47 55.245 90)
+			(at 198.12 55.245 90)
 			(effects
 				(font
@@
 		)
 		(property "Value" "0"
-			(at 209.55 55.245 90)
+			(at 203.2 55.245 90)
 			(effects
 				(font
@@
 		)
 		(property "Footprint" "Resistor_SMD:R_0402_1005Metric_Pad0.72x0.64mm_HandSolder"
-			(at 207.01 57.15 0)
+			(at 200.66 57.15 0)
 			(effects
 				(font
@@
 		)
 		(property "Datasheet" "~"
-			(at 207.01 57.15 0)
+			(at 200.66 57.15 0)
 			(effects
 				(font
@@
 		)
 		(property "Description" ""
-			(at 207.01 57.15 0)
+			(at 200.66 57.15 0)
 			(effects
 				(font
@@
 		)
 		(property "LCSC" "C17168"
-			(at 207.01 57.15 0)
+			(at 200.66 57.15 0)
 			(effects
 				(font
@@
 	(symbol
 		(lib_id "Device:R_Small")
-		(at 213.36 54.61 270)
+		(at 207.01 54.61 270)
 		(mirror x)
 		(unit 1)
@@
 		(dnp no)
 		(property "Reference" "R96"
-			(at 210.82 52.705 90)
+			(at 204.47 52.705 90)
 			(effects
 				(font
@@
 		)
 		(property "Value" "0"
-			(at 215.9 52.705 90)
+			(at 209.55 52.705 90)
 			(effects
 				(font
@@
 		)
 		(property "Footprint" "Resistor_SMD:R_0402_1005Metric_Pad0.72x0.64mm_HandSolder"
-			(at 213.36 54.61 0)
+			(at 207.01 54.61 0)
 			(effects
 				(font
@@
 		)
 		(property "Datasheet" "~"
-			(at 213.36 54.61 0)
+			(at 207.01 54.61 0)
 			(effects
 				(font
@@
 		)
 		(property "Description" ""
-			(at 213.36 54.61 0)
+			(at 207.01 54.61 0)
 			(effects
 				(font
@@
 		)
 		(property "LCSC" "C17168"
-			(at 213.36 54.61 0)
+			(at 207.01 54.61 0)
 			(effects
 				(font
@@
 	)
 	(symbol
+		(lib_id "Connector:TestPoint")
+		(at 288.29 204.47 270)
+		(mirror x)
+		(unit 1)
+		(exclude_from_sim no)
+		(in_bom yes)
+		(on_board yes)
+		(dnp no)
+		(property "Reference" "TP8"
+			(at 294.894 204.47 90)
+			(effects
+				(font
+					(size 1.27 1.27)
+				)
+			)
+		)
+		(property "Value" "TestPoint"
+			(at 296.926 206.248 90)
+			(effects
+				(font
+					(size 1.27 1.27)
+				)
+				(hide yes)
+			)
+		)
+		(property "Footprint" "TestPoint:TestPoint_Pad_1.0x1.0mm"
+			(at 288.29 199.39 0)
+			(effects
+				(font
+					(size 1.27 1.27)
+				)
+				(hide yes)
+			)
+		)
+		(property "Datasheet" "~"
+			(at 288.29 199.39 0)
+			(effects
+				(font
+					(size 1.27 1.27)
+				)
+				(hide yes)
+			)
+		)
+		(property "Description" "test point"
+			(at 288.29 204.47 0)
+			(effects
+				(font
+					(size 1.27 1.27)
+				)
+				(hide yes)
+			)
+		)
+		(pin "1"
+		)
+		(instances
+			(project "ESP32_dual_ESC"
+				(path "/d69d9177-9e27-4190-aaf2-7a8813ea119b/8113d184-5b72-4086-992e-4b0bb4c337ba"
+					(reference "TP8")
+					(unit 1)
+				)
+			)
+		)
+	)
+	(symbol
 		(lib_id "Device:R_Small")
 		(at 330.835 179.07 270)
@@
 					(unit 1)
 				)
+			)
+		)
+	)
+	(symbol
+		(lib_id "Connector:TestPoint")
+		(at 288.29 207.01 270)
+		(mirror x)
+		(unit 1)
+		(exclude_from_sim no)
+		(in_bom yes)
+		(on_board yes)
+		(dnp no)
+		(property "Reference" "TP9"
+			(at 294.894 207.01 90)
+			(effects
+				(font
+					(size 1.27 1.27)
+				)
+			)
+		)
+		(property "Value" "TestPoint"
+			(at 296.926 208.788 90)
+			(effects
+				(font
+					(size 1.27 1.27)
+				)
+				(hide yes)
+			)
+		)
+		(property "Footprint" "TestPoint:TestPoint_Pad_1.0x1.0mm"
+			(at 288.29 201.93 0)
+			(effects
+				(font
+					(size 1.27 1.27)
+				)
+				(hide yes)
+			)
+		)
+		(property "Datasheet" "~"
+			(at 288.29 201.93 0)
+			(effects
+				(font
+					(size 1.27 1.27)
+				)
+				(hide yes)
+			)
+		)
+		(property "Description" "test point"
+			(at 288.29 207.01 0)
+			(effects
+				(font
+					(size 1.27 1.27)
+				)
+				(hide yes)
+			)
+		)
+		(pin "1"
+		)
+		(instances
+			(project "ESP32_dual_ESC"
+				(path "/d69d9177-9e27-4190-aaf2-7a8813ea119b/8113d184-5b72-4086-992e-4b0bb4c337ba"
+					(reference "TP9")
+					(unit 1)
+				)

Commit message: erg
Parts:
- added C33: 1u, Capacitor_SMD:C_0402_1005Metric, symbol Device:C_Small
- added R100, R101, R98, R99: 10k, Resistor_SMD:R_0603_1608Metric, symbol Device:R_Small
- added R102: 2k, Resistor_SMD:R_0402_1005Metric, symbol Device:R_Small
- R95: value 0 -> 10k; footprint Resistor_SMD:R_0402_1005Metric_Pad0.72x0.64mm_HandSolder -> Resistor_SMD:R_0603_1608Metric; LCSC C17168 -> C25804
- U15: LCSC (none) -> C6568
Connections:
- net +VDC is gone; now on net +3V3: R13.1, R13.2
- net +3V3: now also R95.2
- net 1V8: no longer R93.2, R94.2
- net 2V5_RAW: now also U19.5 (+); no longer U13.5 (+)
- net BEMC_Phase_A: now also R81.1; no longer R79.1
- net BEMC_Phase_B: now also R79.1; no longer R80.1
- net BEMC_Phase_C: now also R80.1; no longer R81.1
- net GND: now also C33.1, R102.2, R99.1; no longer R95.1
- net REF_2v5: now also U19.6 (-), U19.7, R98.2; no longer U1.18 (GPIO10/TOUCH10/ADC1_CH9/FSPICS0/FSPIIO4/SUBSPICS0), U13.6 (-), U13.7
- new net: R100.2, R98.1
- new net: R101.2, R95.1, U13.5 (+)
- new net: R101.1, R102.1
- new net 1V81: R93.2, R94.2, U13.6 (-), U13.7
- new net GPIO_10: C33.2, R100.1, R99.2, U1.18 (GPIO10/TOUCH10/ADC1_CH9/FSPICS0/FSPIIO4/SUBSPICS0)
Other:
- moved on the sheet: U13B, U19B
